File: electrical/dronelight.kicad_pcb (KiCad board)
At the start: 2 copper layers, 254 x 71.1 mm, 78 parts, among them J1 SERVO, J2 SERVO, J3 USB_OTG, J4 JTAG, J5 XT60, J6 JST RCY, J7 SAFETY, Q1 DMT6016, Q2 DMT6016, SW1 RESET, SW2 RESET, SW3 RESET, SW4 RESET, U1 LT3755-2-MSE, U2 ATSAMD21G, U3 NCP5501, X1 MTHOLE, X2 MTHOLE, X3 MTHOLE, X4 MTHOLE, X5 MTHOLE, X6 MTHOLE, X7 MTHOLE, X8 MTHOLE

Commit message: Rev 1 redone
Parts:
- removed D10, D11, D12, D13, D14, D5, D6, D7, D8, D9: LED, Libraries:XM-L
- removed D4: B550C, Diodes_SMD:SMC_Handsoldering
- removed FB1: FILTER, Capacitors_SMD:C_0805_HandSoldering
- removed G***: LOGO, Reclaimer_Labs:Reclaimer_Labs
- removed R19: 28.7k, Resistors_SMD:R_0603_HandSoldering
- removed REF**: Symbol_OSHW-Logo_SilkScreen_BIG, Symbols:Symbol_OSHW-Logo_SilkScreen_BIG
- removed SW1, SW2, SW3, SW4: RESET, Libraries:SW_Tact_FSM2JSMA_SMD
- removed X8: MTHOLE, Mounting_Holes:MountingHole_6-5mm
- added C17: 0.1uF, Capacitors_SMD:C_0402, F.Cu at (146.3, 97.0)
- added C18: 0.1uF, Capacitors_SMD:C_0402, F.Cu at (153.7, 101.7)
- added C19: 0.1uF, Capacitors_SMD:C_0402, F.Cu at (156.0, 101.7)
- added C20: 1uF, Capacitors_SMD:C_0603, F.Cu at (148.6, 89.5)
- added C21: 4.7uF, Capacitors_SMD:C_0805, F.Cu at (146.4, 102.4)
- added C22: 4.7uF, Capacitors_SMD:C_0805, F.Cu at (146.4, 100.5)
- added C23: 0.1uF, Capacitors_SMD:C_0402, F.Cu at (146.7, 91.4)
- added C24: DNP, Capacitors_SMD:C_0402, F.Cu at (154.1, 89.7)
- added C25: DNP, Capacitors_SMD:C_0402, F.Cu at (158.5, 91.6)
- added C26: 100pF, Capacitors_SMD:C_0402, F.Cu at (158.5, 90.3)
- added C27: 1uF, Capacitors_SMD:C_0603, F.Cu at (150.9, 89.0)
- added C28: DNP, Capacitors_SMD:C_0603, F.Cu at (158.9, 96.4)
- added C29: 4.7uF, Capacitors_SMD:C_0805, F.Cu at (126.4, 101.6)
- added C30: 0.1uF, Capacitors_SMD:C_0402, F.Cu at (146.4, 88.4)
- added C31: 0.1uF, Capacitors_SMD:C_0402, F.Cu at (160.5, 102.6)
- added L2: 3.3nH, Capacitors_SMD:C_0402, F.Cu at (159.3, 94.5)
- added L3: 3.3nH, Capacitors_SMD:C_0402, F.Cu at (162.3, 94.5)
- added Q3: Photo_Trans, Reclaimer_Labs:Photo_Trans_ALS-PT19-315C, F.Cu at (134.5, 91.4)
- added RT2: 100k, Resistors_SMD:R_0603, F.Cu at (131.4, 91.4)
- added SB1: SB-NC, Reclaimer_Labs:SB-NC, F.Cu at (150.0, 91.4)
- added U4: SPK0415HM4H-B, Reclaimer_Labs:SPK0415HM4H-8, F.Cu at (161.9, 100.3)
- added U5: LPS22HB, Reclaimer_Labs:LGA10R50P2X3_200X200X80, F.Cu at (147.1, 86.2)
- added Y1: 32MHz, Reclaimer_Labs:Crystal_SMD_2016-4pin_2.0x1.6mm, F.Cu at (157.6, 88.0)
- C1: value 0.01uF -> 10uF; footprint Capacitors_SMD:C_0603_HandSoldering -> Capacitors_SMD:C_1206
- C10: value 0.1uF -> 0.8pF; footprint Capacitors_SMD:C_0603_HandSoldering -> Capacitors_SMD:C_0402
- C11: value 0.01uF -> 0.5pF; footprint Capacitors_SMD:C_0603_HandSoldering -> Capacitors_SMD:C_0402
- C12: value 10uF -> 8.2pF; footprint Capacitors_SMD:C_0805_HandSoldering -> Capacitors_SMD:C_0402
- C13: value 0.1uF -> 8.2pF; footprint Capacitors_SMD:C_0603_HandSoldering -> Capacitors_SMD:C_0402
- C14: value 1nF -> 4.7uF; footprint Capacitors_SMD:C_0603_HandSoldering -> Capacitors_SMD:C_0805
- C15: value 4.7uF -> 1uF; footprint Capacitors_SMD:C_0805_HandSoldering -> Capacitors_SMD:C_0603
- C16: value 22uF -> 0.1uF; footprint Capacitors_SMD:C_1210_HandSoldering -> Capacitors_SMD:C_0402
- C2, C3: value 22uF -> 10uF; footprint Capacitors_SMD:C_1210_HandSoldering -> Capacitors_SMD:C_1206
- C4: value 1uF -> 4.7uF; footprint Capacitors_SMD:C_0603_HandSoldering -> Capacitors_SMD:C_1206
- C5: value 0.1uF -> 4.7uF; footprint Capacitors_SMD:C_0603_HandSoldering -> Capacitors_SMD:C_1206
- C6: value 0.1uF -> 0.01uF; footprint Capacitors_SMD:C_0603_HandSoldering -> Capacitors_SMD:C_0603
- C7: value 10uF -> 4.7uF; footprint Capacitors_SMD:C_0805_HandSoldering -> Capacitors_SMD:C_0805
- C8: value 22uF -> 1000pF; footprint Capacitors_SMD:C_1210_HandSoldering -> Capacitors_SMD:C_0603
- C9: value 0.1uF -> 1.2pF; footprint Capacitors_SMD:C_0603_HandSoldering -> Capacitors_SMD:C_0402
- D1: value B550C -> FSV8100V; footprint Diodes_SMD:SMC_Handsoldering -> Reclaimer_Labs:TO-277_3L_Diode
- D2: value B550C -> 1N4148; footprint Diodes_SMD:SMC_Handsoldering -> Diodes_SMD:D_SOD-123
- D3: value RGB_LED_Cree_PLCC4 -> RGB LED 3228 SMD PLCC-4; footprint Libraries:PLCC4-2MM-RGB -> Reclaimer_Labs:PLCC4
- J1: value SERVO -> CONN_01X04; footprint Socket_Strips:Socket_Strip_Straight_1x03 -> Reclaimer_Labs:Header_04x01_2.5mm_RA
- J2: value SERVO -> SAFETY; footprint Socket_Strips:Socket_Strip_Straight_1x03 -> Socket_Strips:Socket_Strip_Straight_1x02_Pitch2.54mm
- J3: value USB_OTG -> ARM_Debug; footprint Libraries:USB_Micro-B_10118194-0001LF -> Reclaimer_Labs:HEADER_SMT_02x05_1.27MM_POL
- J4: value JTAG -> XT30; footprint Libraries:Socket_Strip_Straight_2x10_Shrouded -> Reclaimer_Labs:XT30
- J5: value XT60 -> USB_OTG; footprint Libraries:XT60 -> Reclaimer_Labs:USB_Micro-B_10118194-0001LF
- J6: value JST RCY -> CONN_01X06; footprint Libraries:XT60 -> Socket_Strips:Socket_Strip_Straight_1x06_Pitch2.54mm
- J7: value SAFETY -> CONN_02X06; footprint Socket_Strips:Socket_Strip_Straight_1x02 -> Socket_Strips:Socket_Strip_Straight_2x06_Pitch2.54mm
- L1: footprint Libraries:Inductor_DR127 -> Reclaimer_Labs:Inductor_DR127
- Q1, Q2: footprint Libraries:POWERDI5060-8 -> Reclaimer_Labs:POWERDI5060-8
- R1: value 1k -> 680k; footprint Resistors_SMD:R_0603_HandSoldering -> Resistors_SMD:R_0603
- R10, R12, R13, R14, R9, RT1: footprint Resistors_SMD:R_0603_HandSoldering -> Resistors_SMD:R_0603
- R11: value 10k -> 100k; footprint Resistors_SMD:R_0603_HandSoldering -> Resistors_SMD:R_0603
- R15: value 1k -> 18k; footprint Resistors_SMD:R_0603_HandSoldering -> Resistors_SMD:R_0603
- R16: value 0.005R -> 750k; footprint Resistors_SMD:R_0805_HandSoldering -> Resistors_SMD:R_0603
- R17: value 33mR -> 100k; footprint Resistors_SMD:R_0603_HandSoldering -> Resistors_SMD:R_0603
- R18: value 1M -> 10k; footprint Resistors_SMD:R_0603_HandSoldering -> Resistors_SMD:R_0603
- R2: value 150k -> 825k; footprint Resistors_SMD:R_0603_HandSoldering -> Resistors_SMD:R_0603
- R3: value 1M -> 18k; footprint Resistors_SMD:R_0603_HandSoldering -> Resistors_SMD:R_0603
- R4: value DNP -> 39mR; footprint Resistors_SMD:R_0603_HandSoldering -> Resistors_SMD:R_0603
- R5: value 10k -> 15k; footprint Resistors_SMD:R_0603_HandSoldering -> Resistors_SMD:R_0603
- R6: value 150k -> 100k; footprint Resistors_SMD:R_0603_HandSoldering -> Resistors_SMD:R_0603
- R7: value 1M -> 100k; footprint Resistors_SMD:R_0603_HandSoldering -> Resistors_SMD:R_0603
- R8: value 19.6k -> 0.0005R; footprint Resistors_SMD:R_0603_HandSoldering -> Reclaimer_Labs:CST0612
- U2: value ATSAMD21G -> nrf52840; footprint Housings_QFP:TQFP-48_7x7mm_Pitch0.5mm -> Reclaimer_Labs:AQFN73
- U3: value NCP5501 -> AP2204; footprint Libraries:DPAK3 -> Reclaimer_Labs:SOT89-3
- X1, X2, X3, X4: footprint Mounting_Holes:MountingHole_6-5mm -> Reclaimer_Labs:MountingHole_3.5mm_Pad_Via
- X5, X6, X7: value MTHOLE -> HEATSINK; footprint Mounting_Holes:MountingHole_6-5mm -> Reclaimer_Labs:573100D00010G; moved to B.Cu
- moved X7 161.6 mm to (108.3, 114.3)
- moved X2 150.3 mm to (165.1, 82.5)
- moved J4 116.2 mm to (123.2, 122.6), turned to 0 degrees
- moved R2 114.8 mm to (111.8, 90.8), turned to 180 degrees
- moved J5 113.4 mm to (135.3, 124.5), turned to 0 degrees
- moved R1 104.1 mm to (123.8, 102.2), turned to 270 degrees
- moved X1 101.2 mm to (97.8, 123.2), turned to 90 degrees
- moved X5 94.5 mm to (108.3, 92.7)
- moved X6 89.8 mm to (108.3, 103.5)
- moved C1 87.6 mm to (116.2, 114.3), turned to 90 degrees
- moved J6 85.7 mm to (156.8, 80.5)
- moved X4 78.9 mm to (161.3, 123.2)
- moved R3 71.4 mm to (131.4, 113.0), turned to 180 degrees
- moved J7 70.0 mm to (142.9, 122.6), turned to 90 degrees
- moved R10 69.3 mm to (127.0, 113.7), turned to 270 degrees
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Connections:
- net Net-(Q2-Pad2) renamed /LED Driver Boost/PWMOUT
- net Net-(R9-Pad1) renamed /LED Driver Boost/RT
- C1 pad 1: Net-(C1-Pad1) -> +BATT
- C10 pad 1: +3V3 -> /nrf52840/RF_PIN
- C11 pad 1: Net-(C11-Pad1) -> /nrf52840/RF_MATCHED
- C12 pad 1: +3V3 -> /nrf52840/NRF52_XC2
- C13 pad 1: /~RESET -> /nrf52840/NRF52_XC1
- C14 pad 1: Net-(C14-Pad1) -> +3V3
- C15 pad 1: /INTVCC -> +BATT
- C16 pad 1: Net-(C16-Pad1) -> +3V3
- C2 pad 1: Net-(C2-Pad1) -> +BATT
- C3 pad 1: +3V3 -> +BATT
- C4 pad 1: Net-(C4-Pad1) -> /LED Driver Boost/BOOST_OUT
- C5 pad 1: Net-(C5-Pad1) -> /LED Driver Boost/BOOST_OUT
- C6 pad 1: +3V3 -> /LED Driver Boost/SS
- C7 pad 1: Net-(C5-Pad1) -> /LED Driver Boost/INTVCC
- C8 pad 1: +BATT -> Net-(C8-Pad1)
- C9 pad 1: +3V3 -> GND
- C9 pad 2: GND -> /nrf52840/RF_ANT
- D1 pad 1: Net-(C2-Pad1) -> /LED Driver Boost/BOOST_OUT
- D1 pad 2: +BATT -> /LED Driver Boost/LX
- D2 pad 1: Net-(C2-Pad1) -> +BATT
- D2 pad 2: /USB_VBUS -> VBUS
- J1 pad 1: /SERVO -> /LED Driver Boost/LED_ANODE
- J1 pad 2: GND -> CTRL
- J1 pad 3: /SERVO_PWR -> GND
- J2 pad 1: Net-(J2-Pad1) -> SHDN_L
- J3 pad 1: /USB_VBUS -> +3V3
- J3 pad 2: /USB_DM -> /nrf52840/NRF52_SWDIO
- J3 pad 3: /USB_DP -> GND
- J3 pad 4: Net-(J3-Pad4) -> /nrf52840/NRF52_SWDCLK
- J3 pad 6: Net-(C1-Pad1) -> Net-(J3-Pad6)
- J4 pad 1: +3V3 -> +BATT
- J4 pad 2: Net-(J4-Pad2) -> GND
- J5 pad 1: +BATT -> VBUS
- J5 pad 2: GND -> USB_D_N
- J6 pad 1: +BATT -> GND
- J6 pad 2: GND -> Net-(J6-Pad2)
- J7 pad 1: /~SHDN -> +3V3
- J7 pad 2: GND -> +BATT
- L1 pad 2: Net-(D4-Pad2) -> /LED Driver Boost/LX
- Q1 pad 1: Net-(Q1-Pad1) -> /LED Driver Boost/SENSE
- Q1 pad 3: Net-(D4-Pad2) -> /LED Driver Boost/LX
- Q2 pad 3: Net-(D14-Pad1) -> /LED Driver Boost/LED_CATHODE
- R1 pad 1: +3V3 -> SHDN_L
- R1 pad 2: /SWDCLK -> +BATT
- R10 pad 1: +3V3 -> Net-(R10-Pad1)
- R10 pad 2: /~RESET -> Net-(C8-Pad1)
- R11 pad 1: Net-(R11-Pad1) -> +3V3
- R11 pad 2: Net-(C14-Pad1) -> /nrf52840/NRF52_RESET_L
- R12 pad 1: /~RESET -> Net-(D3-Pad4)
- R12 pad 2: Net-(R12-Pad2) -> RGB_RED
- R13 pad 1: /RGB_BLU -> Net-(D3-Pad3)
- R13 pad 2: Net-(D3-Pad2) -> RGB_GRN
- R14 pad 1: Net-(D3-Pad3) -> Net-(D3-Pad2)
- R14 pad 2: /RGB_GRN -> RGB_BLU
- R15 pad 1: Net-(D3-Pad4) -> /nrf52840/BOARD_TEMP
- R15 pad 2: /RGB_RED -> +3V3
- R16 pad 1: Net-(Q1-Pad1) -> /nrf52840/VBATT_MEAS
- R16 pad 2: GND -> +BATT
- R17 pad 1: Net-(D5-Pad2) -> GND
- R17 pad 2: Net-(C16-Pad1) -> /nrf52840/VBATT_MEAS
- R18 pad 1: Net-(R18-Pad1) -> GND
- R18 pad 2: Net-(C16-Pad1) -> PHOTO_SENSE
- R2 pad 1: /SWDIO -> /LED Driver Boost/FB
- R2 pad 2: +3V3 -> /LED Driver Boost/BOOST_OUT
- R3 pad 1: GND -> /LED Driver Boost/VREF
- R3 pad 2: Net-(C1-Pad1) -> CTRL
- R4 pad 1: +3V3 -> /LED Driver Boost/LED_ANODE
- R4 pad 2: /SERVO_PWR -> /LED Driver Boost/BOOST_OUT
- R5 pad 1: +3V3 -> /LED Driver Boost/FB
- R5 pad 2: /~OPENLED -> GND
- R6 pad 1: /~SHDN -> GND
- R6 pad 2: GND -> SHDN_L
- R7 pad 1: +BATT -> +3V3
- R7 pad 2: /~SHDN -> OPENLED_L
- R8 pad 1: Net-(R8-Pad1) -> /LED Driver Boost/SENSE
- R8 pad 2: /CTRL -> GND
- RT1 pad 1: GND -> CTRL
- RT1 pad 2: /CTRL -> GND
- U1 pad 10: Net-(C11-Pad1) -> /LED Driver Boost/SS
- U1 pad 12: /~SHDN -> SHDN_L
- U1 pad 13: /INTVCC -> /LED Driver Boost/INTVCC
- U1 pad 15: Net-(Q1-Pad1) -> /LED Driver Boost/SENSE
- U1 pad 2: Net-(R18-Pad1) -> /LED Driver Boost/FB
- U1 pad 3: Net-(D5-Pad2) -> /LED Driver Boost/LED_ANODE
- U1 pad 4: Net-(C16-Pad1) -> /LED Driver Boost/BOOST_OUT
- U1 pad 5: Net-(R11-Pad1) -> Net-(R10-Pad1)
- U1 pad 6: /CTRL -> CTRL
- U1 pad 7: Net-(R8-Pad1) -> /LED Driver Boost/VREF
- U1 pad 8: /PWMIN -> PWMIN
- U1 pad 9: /~OPENLED -> OPENLED_L
- U3 pad 1: Net-(C2-Pad1) -> +BATT
- X1 pad 1: Net-(X1-Pad1) -> GND
- X2 pad 1: Net-(X2-Pad1) -> GND
- X3 pad 1: Net-(X3-Pad1) -> GND
- X4 pad 1: Net-(X4-Pad1) -> GND
- X5 pad 1: Net-(X5-Pad1) -> GND
- X6 pad 1: Net-(X6-Pad1) -> GND
- X7 pad 1: Net-(X7-Pad1) -> GND
Routing:
- net /THERMAL: track 426.3 -> 0.00 mm, vias 280 -> 0
- net GND: track 211.1 -> 624.8 mm, vias 63 -> 313
- net Net-(D14-Pad1): track 198.0 -> 0.00 mm, vias 24 -> 0
- net +BATT: track 279.6 -> 90.3 mm, vias 16 -> 2
- net Net-(D5-Pad2): track 169.5 -> 0.00 mm
- net /USB_VBUS: track 102.2 -> 0.00 mm, vias 2 -> 0
- net /CTRL: track 88.4 -> 0.00 mm, vias 4 -> 0
- net /SWDIO: track 84.6 -> 0.00 mm, vias 2 -> 0
- net CTRL: track 0.00 -> 84.5 mm, vias 0 -> 2
- net /~OPENLED: track 80.8 -> 0.00 mm, vias 4 -> 0
- net /SWDCLK: track 80.4 -> 0.00 mm, vias 2 -> 0
- net Net-(R12-Pad2): track 80.0 -> 0.00 mm, vias 2 -> 0
- net /LED Driver Boost/BOOST_OUT: track 0.00 -> 78.9 mm, vias 0 -> 2
- net /~SHDN: track 77.1 -> 0.00 mm, vias 1 -> 0
- net /~RESET: track 62.4 -> 0.00 mm, vias 2 -> 0
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- added copper zone on F.Cu, net /LED Driver Boost/BOOST_OUT
- added copper zone on F.Cu, net /LED Driver Boost/LED_ANODE
- added copper zone on F.Cu, net /LED Driver Boost/LED_CATHODE
- added copper zone on F.Cu, net /LED Driver Boost/LX
- added copper zone on F.Cu, net /LED Driver Boost/SENSE
- removed copper zone on B.Cu, net +BATT
- removed copper zone on B.Cu, net /THERMAL
- removed copper zone on F.Cu, net /THERMAL
- removed copper zone on F.Cu, net /USB_VBUS
- removed copper zone on F.Cu, net Net-(C16-Pad1)
- removed copper zone on F.Cu, net Net-(C2-Pad1)
- removed copper zone on F.Cu, net Net-(D10-Pad1)
- removed copper zone on F.Cu, net Net-(D10-Pad2)
- removed copper zone on F.Cu, net Net-(D11-Pad1)
- removed copper zone on F.Cu, net Net-(D12-Pad1)
- removed copper zone on F.Cu, net Net-(D13-Pad1)
- removed copper zone on B.Cu, net Net-(D14-Pad1)
- removed copper zone on F.Cu, net Net-(D14-Pad1)
- removed copper zone on F.Cu, net Net-(D4-Pad2)
- removed copper zone on F.Cu, net Net-(D5-Pad1)
- removed copper zone on F.Cu, net Net-(D5-Pad2)
- removed copper zone on F.Cu, net Net-(D6-Pad1)
- removed copper zone on F.Cu, net Net-(D7-Pad1)
- removed copper zone on F.Cu, net Net-(D8-Pad1)
- removed copper zone on F.Cu, net Net-(Q1-Pad1)
Other:
- board size 254 x 71.1 mm -> 83.2 x 48.3 mm
- net class Default: clearance 0.1524 -> 0.126746; trace_width 0.1524 -> 0.127; via_dia 0.6858 -> 0.6096; via_drill 0.3302 -> 0.3048
- net class Thicker: clearance 0.1524 -> 0.126746; via_dia 0.6858 -> 0.6096; via_drill 0.3302 -> 0.3048
- rule trace_clearance: 0.1524 -> 0.126746
- rule trace_min: 0.1524 -> 0.126746
- rule via_min_drill: 0.3302 -> 0.3048
- rule via_min_size: 0.6858 -> 0.6096
- board text added: "+3V3"
- board text added: "0.13"
- board text added: "0.15"
- board text added: "0.20"
- board text added: "0.22"
- board text added: "0.24"
- board text added: "1.00"
- board text added: "1.02"
- board text added: "1.04"
- board text added: "1.06"
- board text added: "12-24 VDC 150 W"
- board text added: "3V3"
- board text added: "BATT"
- board text added: "BLK"
- board text added: "C"
- board text added: "CTS"
- board text added: "DEBUG"
- board text added: "Dronelight Rev 2 Reclaimer Labs"
- board text added: "E"
- board text added: "GRN"
- board text added: "RTS"
- board text added: "SHDN"
- board text removed: "10-25VDC 10A MAX"
- board text removed: "2 LAYER 0.031 inch Thickness 2 oz copper 6/6 mil Trace/Space 13 mil min hole size 7 mil min ring"
- board text removed: "DO NOT STARE AT LEDs DO NOT TOUCH LEDs"
- board text removed: "Drone Light Rev 1 - 08 Mar 2016 Reclaimer Labs http://reclaimerlabs.com"
- board text removed: "JTAG"
- board text removed: "POWER"
- board text removed: "PWR"
- board text removed: "SERVO IN"
- board text removed: "SIG"
- board text removed: "USE ONE XT60 MAX"
- board text removed: "USE ONE XT60 ONLY"
- board text removed: "WARNING! THESE LEDs ARE REALLY BRIGHT AND HOT - 85C / 185F"
- board text removed: "XT60"
