File: electrical/dronelight.sch (KiCad schematic (older format))
At the start: 76 parts, among them J1 SERVO, J2 SERVO, J3 USB_OTG, J4 JTAG, J5 XT60, J6 JST RCY, J7 SAFETY, Q1 DMT6016, Q2 DMT6016, SW1 RESET, SW2 RESET, SW3 RESET, SW4 RESET, U1 LT3755-2-MSE, U2 ATSAMD21G, U3 NCP5501, X1 MTHOLE, X2 MTHOLE, X3 MTHOLE, X4 MTHOLE, X5 MTHOLE, X6 MTHOLE, X7 MTHOLE, X8 MTHOLE

Commit message: Rev 1 redone
Parts:
- removed C1, C11: 0.01uF, Capacitors_SMD:C_0603_HandSoldering, symbol C
- removed C10, C13, C5, C6, C9: 0.1uF, Capacitors_SMD:C_0603_HandSoldering, symbol C
- removed C12, C7: 10uF, Capacitors_SMD:C_0805_HandSoldering, symbol C
- removed C14: 1nF, Capacitors_SMD:C_0603_HandSoldering, symbol C
- removed C15: 4.7uF, Capacitors_SMD:C_0805_HandSoldering, symbol C
- removed C16, C2, C3, C8: 22uF, Capacitors_SMD:C_1210_HandSoldering, symbol C
- removed C4: 1uF, Capacitors_SMD:C_0603_HandSoldering, symbol C
- removed D1, D2, D4: B550C, Diodes_SMD:SMC_Handsoldering, symbol D_Schottky
- removed D10, D11, D12, D13, D14, D5, D6, D7, D8, D9: LED, Libraries:XM-L, symbol Led_Small
- removed D3: RGB_LED_Cree_PLCC4, Libraries:PLCC4-2MM-RGB, symbol RGB_LED_Cree_PLCC4
- removed FB1: FILTER, Capacitors_SMD:C_0805_HandSoldering, symbol FILTER
- removed J1, J2: SERVO, Socket_Strips:Socket_Strip_Straight_1x03, symbol CONN_01X03
- removed J3: USB_OTG, Libraries:USB_Micro-B_10118194-0001LF, symbol USB_OTG
- removed J4: JTAG, Libraries:Socket_Strip_Straight_2x10_Shrouded, symbol CONN_02X10
- removed J5: XT60, Libraries:XT60, symbol CONN_01X02
- removed J6: JST RCY, Libraries:XT60, symbol CONN_01X02
- removed J7: SAFETY, Socket_Strips:Socket_Strip_Straight_1x02, symbol CONN_01X02
- removed L1: 22uH, Libraries:Inductor_DR127, symbol INDUCTOR
- removed Q1, Q2: DMT6016, Libraries:POWERDI5060-8, symbol Q_NMOS_SGD
- removed R1, R12, R13, R14, R15: 1k, Resistors_SMD:R_0603_HandSoldering, symbol R
- removed R10, R11, R5: 10k, Resistors_SMD:R_0603_HandSoldering, symbol R
- removed R16: 0.005R, Resistors_SMD:R_0805_HandSoldering, symbol R
- removed R17: 33mR, Resistors_SMD:R_0603_HandSoldering, symbol R
- removed R18, R3, R7: 1M, Resistors_SMD:R_0603_HandSoldering, symbol R
- removed R19, R9: 28.7k, Resistors_SMD:R_0603_HandSoldering, symbol R
- removed R2, R6: 150k, Resistors_SMD:R_0603_HandSoldering, symbol R
- removed R4: DNP, Resistors_SMD:R_0603_HandSoldering, symbol R
- removed R8: 19.6k, Resistors_SMD:R_0603_HandSoldering, symbol R
- removed RT1: 100k, Resistors_SMD:R_0603_HandSoldering, symbol PTC
- removed SW1, SW2, SW3, SW4: RESET, Libraries:SW_Tact_FSM2JSMA_SMD, symbol SW_Tact_NO
- removed U1: LT3755-2-MSE, Housings_SSOP:MSOP-16-1EP_3x4mm_Pitch0.5mm, symbol LT3755-2-MSE
- removed U2: ATSAMD21G, Housings_QFP:TQFP-48_7x7mm_Pitch0.5mm, symbol ATSAMD21G
- removed U3: NCP5501, Libraries:DPAK3, symbol NCP5501
- removed X1, X2, X3, X4, X5, X6, X7, X8: MTHOLE, Mounting_Holes:MountingHole_6-5mm, symbol MTHOLE
Connections:
- no-connect marks 17 -> 0
Other:
- note removed: "375kHz"
- note removed: "Big\nHoles"
- note removed: "Remove\nbefore\nflight!"
- note removed: "Vout = 44.8 V max"
